File: rollxoxo-shim.kicad_sch (KiCad schematic)
At the start: 70 parts, among them J1 USB_C_Receptacle_USB2.0_14P, J2 Conn_01x02, J3 Conn_01x10, J4 Conn_01x01, J5 Conn_01x10, J6 Conn_01x03, J7 Conn_01x01, SW1 SW_Push, SW2 SW_Push, U1 SN74LV1T125DBV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

Commit message: pcb: initial rough placement
Connections:
- net +5V: now also J3.7 (Pin_7), J5.7 (Pin_7); no longer J3.4 (Pin_4), J5.4 (Pin_4)
- net DOWN_BTN: now also J3.10 (Pin_10), J5.10 (Pin_10); no longer J3.1 (Pin_1), J5.1 (Pin_1)
- net STOP_BTN: now also J3.6 (Pin_6), J5.6 (Pin_6); no longer J3.5 (Pin_5), J5.5 (Pin_5)
- net UP_BTN: now also J3.1 (Pin_1), J5.1 (Pin_1); no longer J3.10 (Pin_10), J5.10 (Pin_10)
- new net: J3.4 (Pin_4), J5.4 (Pin_4)
- new net: J3.5 (Pin_5), J5.5 (Pin_5)
Changed lines of the file:
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@@
 	)
 	(symbol
+		(lib_id "Connector_Generic:Conn_01x10")
+		(at 105.41 113.03 0)
+		(mirror x)
+		(unit 1)
+		(body_style 1)
+		(exclude_from_sim no)
+		(in_bom no)
+		(on_board yes)
+		(in_pos_files yes)
+		(dnp no)
+		(property "Reference" "J5"
+			(at 107.95 111.7601 0)
+			(show_name no)
+			(do_not_autoplace no)
+			(effects
+				(font
+					(size 1.27 1.27)
+				)
+				(justify left)
+			)
+		)
+		(property "Value" "Conn_01x10"
+			(at 107.95 110.4901 0)
+			(hide yes)
+			(show_name no)
+			(do_not_autoplace no)
+			(effects
+				(font
+					(size 1.27 1.27)
+				)
+				(justify left)
+			)
+		)
+		(property "Footprint" "Connector_PinHeader_2.54mm:PinHeader_1x10_P2.54mm_Horizontal"
+			(at 105.41 113.03 0)
+			(hide yes)
+			(show_name no)
+			(do_not_autoplace no)
+			(effects
+				(font
+					(size 1.27 1.27)
+				)
+			)
+		)
+		(property "Datasheet" ""
+			(at 105.41 113.03 0)
+			(hide yes)
+			(show_name no)
+			(do_not_autoplace no)
+			(effects
+				(font
+					(size 1.27 1.27)
+				)
+			)
+		)
+		(property "Description" "Generic connector, single row, 01x10, script generated (kicad-library-utils/schlib/autogen/connector/)"
+			(at 105.41 113.03 0)
+			(hide yes)
+			(show_name no)
+			(do_not_autoplace no)
+			(effects
+				(font
+					(size 1.27 1.27)
+				)
+			)
+		)
+		(pin "9"
+		)
+		(pin "6"
+		)
+		(pin "8"
+		)
+		(pin "3"
+		)
+		(pin "5"
+		)
+		(pin "2"
+		)
+		(pin "10"
+		)
+		(pin "7"
+		)
+		(pin "4"
+		)
+		(pin "1"
+		)
+		(instances
+			(project "rollxoxo-shim"
+				(path "/a7ed83d6-0dbd-4a58-9db2-84a345940fc7"
+					(reference "J5")
+					(unit 1)
+				)
+			)
+		)
+	)
+	(symbol
 		(lib_id "power:GND")
 		(at 171.45 66.04 0)
@@
 	)
 	(symbol
-		(lib_id "Connector_Generic:Conn_01x10")
-		(at 105.41 110.49 0)
-		(unit 1)
-		(body_style 1)
-		(exclude_from_sim no)
-		(in_bom no)
-		(on_board yes)
-		(in_pos_files yes)
-		(dnp no)
-		(property "Reference" "J5"
-			(at 107.95 111.7599 0)
-			(show_name no)
-			(do_not_autoplace no)
-			(effects
-				(font
-					(size 1.27 1.27)
-				)
-				(justify left)
-			)
-		)
-		(property "Value" "Conn_01x10"
-			(at 107.95 113.0299 0)
-			(hide yes)
-			(show_name no)
-			(do_not_autoplace no)
-			(effects
-				(font
-					(size 1.27 1.27)
-				)
-				(justify left)
-			)
-		)
-		(property "Footprint" "Connector_PinHeader_2.54mm:PinHeader_1x10_P2.54mm_Horizontal"
-			(at 105.41 110.49 0)
-			(hide yes)
-			(show_name no)
-			(do_not_autoplace no)
-			(effects
-				(font
-					(size 1.27 1.27)
-				)
-			)
-		)
-		(property "Datasheet" ""
-			(at 105.41 110.49 0)
-			(hide yes)
-			(show_name no)
-			(do_not_autoplace no)
-			(effects
-				(font
-					(size 1.27 1.27)
-				)
-			)
-		)
-		(property "Description" "Generic connector, single row, 01x10, script generated (kicad-library-utils/schlib/autogen/connector/)"
-			(at 105.41 110.49 0)
-			(hide yes)
-			(show_name no)
-			(do_not_autoplace no)
-			(effects
-				(font
-					(size 1.27 1.27)
-				)
-			)
-		)
-		(pin "9"
-		)
-		(pin "6"
-		)
-		(pin "8"
-		)
-		(pin "3"
-		)
-		(pin "5"
-		)
-		(pin "2"
-		)
-		(pin "10"
-		)
-		(pin "7"
-		)
-		(pin "4"
-		)
-		(pin "1"
-		)
-		(instances
-			(project "rollxoxo-shim"
-				(path "/a7ed83d6-0dbd-4a58-9db2-84a345940fc7"
-					(reference "J5")
-					(unit 1)
-				)
-			)
-		)
-	)
-	(symbol
 		(lib_id "power:GND")
 		(at 229.87 31.75 0)
@@
 	)
 	(symbol
+		(lib_id "Connector_Generic:Conn_01x10")
+		(at 81.28 113.03 180)
+		(unit 1)
+		(body_style 1)
+		(exclude_from_sim no)
+		(in_bom no)
+		(on_board yes)
+		(in_pos_files yes)
+		(dnp no)
+		(property "Reference" "J3"
+			(at 78.74 111.7601 0)
+			(show_name no)
+			(do_not_autoplace no)
+			(effects
+				(font
+					(size 1.27 1.27)
+				)
+				(justify left)
+			)
+		)
+		(property "Value" "Conn_01x10"
+			(at 78.74 110.4901 0)
+			(hide yes)
+			(show_name no)
+			(do_not_autoplace no)
+			(effects
+				(font
+					(size 1.27 1.27)
+				)
+				(justify left)
+			)
+		)
+		(property "Footprint" "Connector_PinSocket_2.54mm:PinSocket_1x10_P2.54mm_Horizontal"
+			(at 81.28 113.03 0)
+			(hide yes)
+			(show_name no)
+			(do_not_autoplace no)
+			(effects
+				(font
+					(size 1.27 1.27)
+				)
+			)
+		)
+		(property "Datasheet" ""
+			(at 81.28 113.03 0)
+			(hide yes)
+			(show_name no)
+			(do_not_autoplace no)
+			(effects
+				(font
+					(size 1.27 1.27)
+				)
+			)
+		)
+		(property "Description" "Generic connector, single row, 01x10, script generated (kicad-library-utils/schlib/autogen/connector/)"
+			(at 81.28 113.03 0)
+			(hide yes)
+			(show_name no)
+			(do_not_autoplace no)
+			(effects
+				(font
+					(size 1.27 1.27)
+				)
+			)
+		)
+		(pin "9"
+		)
+		(pin "6"
+		)
+		(pin "8"
+		)
+		(pin "3"
+		)
+		(pin "5"
+		)
+		(pin "2"
+		)
+		(pin "10"
+		)
+		(pin "7"
+		)
+		(pin "4"
+		)
+		(pin "1"
+		)
+		(instances
+			(project "rollxoxo-shim"
+				(path "/a7ed83d6-0dbd-4a58-9db2-84a345940fc7"
+					(reference "J3")
+					(unit 1)
+				)
+			)
+		)
+	)
+	(symbol
 		(lib_id "power:GND")
 		(at 133.35 190.5 0)
@@
 					(unit 1)
 				)
-			)
-		)
-	)
-	(symbol
-		(lib_id "Connector_Generic:Conn_01x10")
-		(at 81.28 110.49 0)
-		(mirror y)
-		(unit 1)
-		(body_style 1)
-		(exclude_from_sim no)
-		(in_bom no)
-		(on_board yes)
-		(in_pos_files yes)
-		(dnp no)
-		(property "Reference" "J3"
-			(at 78.74 111.7599 0)
-			(show_name no)
-			(do_not_autoplace no)
-			(effects
-				(font
-					(size 1.27 1.27)
-				)
-				(justify left)
-			)
-		)
-		(property "Value" "Conn_01x10"
-			(at 78.74 113.0299 0)
-			(hide yes)
-			(show_name no)
-			(do_not_autoplace no)
-			(effects
-				(font
-					(size 1.27 1.27)
-				)
-				(justify left)
-			)
-		)
-		(property "Footprint" "Connector_PinSocket_2.54mm:PinSocket_1x10_P2.54mm_Horizontal"
-			(at 81.28 110.49 0)
-			(hide yes)
-			(show_name no)
-			(do_not_autoplace no)
-			(effects
-				(font
-					(size 1.27 1.27)
-				)
-			)
-		)
-		(property "Datasheet" ""
-			(at 81.28 110.49 0)
-			(hide yes)
-			(show_name no)
-			(do_not_autoplace no)
-			(effects
-				(font
-					(size 1.27 1.27)
-				)
-			)
-		)
-		(property "Description" "Generic connector, single row, 01x10, script generated (kicad-library-utils/schlib/autogen/connector/)"
-			(at 81.28 110.49 0)
-			(hide yes)
-			(show_name no)
-			(do_not_autoplace no)
-			(effects
-				(font
-					(size 1.27 1.27)
-				)
-			)
-		)
-		(pin "9"
-		)
-		(pin "6"
-		)
-		(pin "8"
-		)
-		(pin "3"
-		)
-		(pin "5"
-		)
-		(pin "2"
-		)
-		(pin "10"
-		)
-		(pin "7"
-		)
-		(pin "4"
-		)
-		(pin "1"
-		)
-		(instances
-			(project "rollxoxo-shim"
-				(path "/a7ed83d6-0dbd-4a58-9db2-84a345940fc7"
-					(reference "J3")
-					(unit 1)
-				)

Commit message: pcb: refine layout
Parts:
- removed TP5, TP6: TestPoint, TestPoint:TestPoint_Pad_D1.0mm, symbol Connector:TestPoint
- J2: footprint Connector_JST:JST_XH_S2B-XH-A_1x02_P2.50mm_Horizontal -> Connector_JST:JST_XH_B2B-XH-A_1x02_P2.50mm_Vertical
Connections:
- net GND: now also J1.SH (SHIELD); no longer J1.S1 (SHIELD)
- no-connect marks 37 -> 39
Changed lines of the file:
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@@
 	)
 	(no_connect
+		(at 250.19 66.04)
+	)
+	(no_connect
 		(at 184.15 116.84)
 	)
@@
 	)
 	(no_connect
+		(at 250.19 68.58)
+	)
+	(no_connect
 		(at 250.19 124.46)
 	)
@@
 	(wire
 		(pts
-			(xy 251.46 68.58) (xy 250.19 68.58)
-		)
-		(stroke
-			(width 0)
-			(type default)
-		)
-	)
-	(wire
-		(pts
 			(xy 85.09 171.45) (xy 85.09 170.18)
 		)
@@
 	(wire
 		(pts
-			(xy 251.46 66.04) (xy 250.19 66.04)
-		)
-		(stroke
-			(width 0)
-			(type default)
-		)
-	)
-	(wire
-		(pts
 			(xy 100.33 179.07) (xy 100.33 177.8)
 		)
@@
 		(pin "A1"
 		)
-		(pin "S1"
+		(pin "SH"
 		)
 		(pin "B9"
@@
 	)
 	(symbol
-		(lib_id "Connector:TestPoint")
-		(at 251.46 66.04 270)
-		(unit 1)
-		(body_style 1)
-		(exclude_from_sim no)
-		(in_bom no)
-		(on_board yes)
-		(in_pos_files yes)
-		(dnp no)
-		(property "Reference" "TP5"
-			(at 256.286 66.04 90)
-			(show_name no)
-			(do_not_autoplace no)
-			(effects
-				(font
-					(size 1.27 1.27)
-				)
-				(justify left)
-			)
-		)
-		(property "Value" "TestPoint"
-			(at 253.4921 68.58 0)
-			(hide yes)
-			(show_name no)
-			(do_not_autoplace no)
-			(effects
-				(font
-					(size 1.27 1.27)
-				)
-				(justify left)
-			)
-		)
-		(property "Footprint" "TestPoint:TestPoint_Pad_D1.0mm"
-			(at 251.46 71.12 0)
-			(hide yes)
-			(show_name no)
-			(do_not_autoplace no)
-			(effects
-				(font
-					(size 1.27 1.27)
-				)
-			)
-		)
-		(property "Datasheet" ""
-			(at 251.46 71.12 0)
-			(hide yes)
-			(show_name no)
-			(do_not_autoplace no)
-			(effects
-				(font
-					(size 1.27 1.27)
-				)
-			)
-		)
-		(property "Description" "test point"
-			(at 251.46 66.04 0)
-			(hide yes)
-			(show_name no)
-			(do_not_autoplace no)
-			(effects
-				(font
-					(size 1.27 1.27)
-				)
-			)
-		)
-		(pin "1"
-		)
-		(instances
-			(project "rollxoxo-shim"
-				(path "/a7ed83d6-0dbd-4a58-9db2-84a345940fc7"
-					(reference "TP5")
-					(unit 1)
-				)
-			)
-		)
-	)
-	(symbol
 		(lib_id "Device:C")
 		(at 191.77 35.56 0)
@@
 			)
 		)
-		(property "Footprint" "Connector_JST:JST_XH_S2B-XH-A_1x02_P2.50mm_Horizontal"
+		(property "Footprint" "Connector_JST:JST_XH_B2B-XH-A_1x02_P2.50mm_Vertical"
 			(at 78.74 170.18 0)
 			(hide yes)
@@
 					(unit 1)
 				)
-			)
-		)
-	)
-	(symbol
-		(lib_id "Connector:TestPoint")
-		(at 251.46 68.58 270)
-		(unit 1)
-		(body_style 1)
-		(exclude_from_sim no)
-		(in_bom no)
-		(on_board yes)
-		(in_pos_files yes)
-		(dnp no)
-		(property "Reference" "TP6"
-			(at 256.286 68.58 90)
-			(show_name no)
-			(do_not_autoplace no)
-			(effects
-				(font
-					(size 1.27 1.27)
-				)
-				(justify left)
-			)
-		)
-		(property "Value" "TestPoint"
-			(at 253.4921 71.12 0)
-			(hide yes)
-			(show_name no)
-			(do_not_autoplace no)
-			(effects
-				(font
-					(size 1.27 1.27)
-				)
-				(justify left)
-			)
-		)
-		(property "Footprint" "TestPoint:TestPoint_Pad_D1.0mm"
-			(at 251.46 73.66 0)
-			(hide yes)
-			(show_name no)
-			(do_not_autoplace no)
-			(effects
-				(font
-					(size 1.27 1.27)
-				)
-			)
-		)
-		(property "Datasheet" ""
-			(at 251.46 73.66 0)
-			(hide yes)
-			(show_name no)
-			(do_not_autoplace no)
-			(effects
-				(font
-					(size 1.27 1.27)
-				)
-			)
-		)
-		(property "Description" "test point"
-			(at 251.46 68.58 0)
-			(hide yes)
-			(show_name no)
-			(do_not_autoplace no)
-			(effects
-				(font
-					(size 1.27 1.27)
-				)
-			)
-		)
-		(pin "1"
-		)
-		(instances
-			(project "rollxoxo-shim"
-				(path "/a7ed83d6-0dbd-4a58-9db2-84a345940fc7"
-					(reference "TP6")
-					(unit 1)
-				)

Commit message: pcb: reorganize programmable gpios
Connections:
- net FLASH: now also U6.6 (GPIO1/ADC1_CH0); no longer U6.14 (GPIO9/ADC1_CH8)
Changed lines of the file:
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@@
-	)
-	(no_connect
-		(at 250.19 83.82)
 	)
 	(no_connect
@@
 	)
 	(no_connect
+		(at 250.19 104.14)
+	)
+	(no_connect
 		(at 250.19 111.76)
 	)
@@
 	(wire
 		(pts
-			(xy 260.35 96.52) (xy 250.19 96.52)
+			(xy 259.08 96.52) (xy 250.19 96.52)
+		)
+		(stroke
+			(width 0)
+			(type default)
+		)
+	)
+	(wire
+		(pts
+			(xy 259.08 83.82) (xy 250.19 83.82)
 		)
 		(stroke
@@
 	(wire
 		(pts
-			(xy 260.35 91.44) (xy 250.19 91.44)
+			(xy 259.08 91.44) (xy 250.19 91.44)
 		)
 		(stroke
@@
 	(wire
 		(pts
-			(xy 260.35 109.22) (xy 250.19 109.22)
+			(xy 259.08 109.22) (xy 250.19 109.22)
 		)
 		(stroke
@@
 	(wire
 		(pts
-			(xy 260.35 104.14) (xy 250.19 104.14)
-		)
-		(stroke
-			(width 0)
-			(type default)
-		)
-	)
-	(wire
-		(pts
 			(xy 100.33 143.51) (xy 100.33 142.24)
 		)
@@
 	(wire
 		(pts
-			(xy 260.35 106.68) (xy 250.19 106.68)
+			(xy 259.08 106.68) (xy 250.19 106.68)
 		)
 		(stroke
@@
 	(wire
 		(pts
-			(xy 260.35 93.98) (xy 250.19 93.98)
+			(xy 259.08 93.98) (xy 250.19 93.98)
 		)
 		(stroke
@@
 	(wire
 		(pts
-			(xy 260.35 101.6) (xy 250.19 101.6)
+			(xy 259.08 101.6) (xy 250.19 101.6)
 		)
 		(stroke
@@
 		)
 	)
-	(label "FLASH"
-		(at 260.35 104.14 180)
-		(effects
-			(font
-				(size 1.27 1.27)
-			)
-			(justify right bottom)
-		)
-	)
 	(label "XTAL_N"
 		(at 105.41 142.24 180)
@@
 		)
 	)
+	(label "FLASH"
+		(at 259.08 83.82 180)
+		(effects
+			(font
+				(size 1.27 1.27)
+			)
+			(justify right bottom)
+		)
+	)
 	(label "UP_BTN"
 		(at 59.69 125.73 180)
@@
 	)
 	(label "REED_B"
-		(at 260.35 109.22 180)
+		(at 259.08 109.22 180)
 		(effects
 			(font
@@
 	)
 	(label "LIGHT"
-		(at 260.35 101.6 180)
+		(at 259.08 101.6 180)
 		(effects
 			(font
@@
 	)
 	(label "DOWN"
-		(at 260.35 91.44 180)
+		(at 259.08 91.44 180)
 		(effects
 			(font
@@
 	)
 	(label "REED_A"
-		(at 260.35 106.68 180)
+		(at 259.08 106.68 180)
 		(effects
 			(font
@@
 	)
 	(label "STOP"
-		(at 260.35 93.98 180)
+		(at 259.08 93.98 180)
 		(effects
 			(font
@@
 	)
 	(label "UP"
-		(at 260.35 96.52 180)
-		(effects
-			(font
+		(at 259.08 96.52 180)
+		(effects
+			(font

Commit message: pcb: route gpios
Connections:
- net DOWN: now also U6.19 (GPIO14/ADC2_CH3); no longer U6.9 (GPIO4/ADC1_CH3)
- net FLASH: now also U6.12 (GPIO7/ADC1_CH6); no longer U6.6 (GPIO1/ADC1_CH0)
- net LIGHT: now also U6.14 (GPIO9/ADC1_CH8); no longer U6.13 (GPIO8/ADC1_CH7)
- net REED_A: now also U6.6 (GPIO1/ADC1_CH0); no longer U6.15 (GPIO10/ADC1_CH9)
- net REED_B: now also U6.7 (GPIO2/ADC1_CH1); no longer U6.16 (GPIO11/ADC2_CH0)
- net STOP: now also U6.17 (GPIO12/ADC2_CH1); no longer U6.10 (GPIO5/ADC1_CH4)
- net UP: now also U6.15 (GPIO10/ADC1_CH9); no longer U6.11 (GPIO6/ADC1_CH5)

Commit message: schem/pcb: add tooling holes
Parts:
- added H5, H6, H7: MountingHole, MountingHole:ToolingHole_1.152mm, symbol Mechanical:MountingHole
Other:
- note added: "SMT assembly"
